Commit message: Added wheels

File: exc_description/urdf/exc.xacro (robot description, xacro)
@@ -5,4 +5,47 @@
   <xacro:property name="base_length" value="${58*itom}"/> <!-- Max val: 50" bare minimum -->
   <xacro:property name="base_height" value="${2*itom}"/> <!-- BS'd this number, total random guess -->
+  <xacro:property name="wheel_radius" value="${16*itom}"/>
+  <xacro:property name="wheel_width" value="${6*itom}"/>
+  <xacro:include filename="$(find exc_description)/urdf/exc.gazebo" />
+  <!-- A macro for creating a wheel with a link, joint, and transmission -->
+  <xacro:macro name="wheel" params="name fb lr">
+    <link name="${name}">
+      <visual>
+        <geometry>
+          <cylinder radius="${wheel_radius}" length="${wheel_width}" />
+        </geometry>
+        <origin rpy="${pi/2} 0 0" />
+      </visual>
+      <collision>
+        <geometry>
+          <cylinder radius="${wheel_radius}" length="${wheel_width}" />
+        </geometry>
+        <origin rpy="${pi/2} 0 0" />
+      </collision>
+      <inertial>
+        <origin xyz="0 ${wheel_width/2} 0" rpy="0 0 0"/>
+        <mass value="500"/> <!-- TODO: Update with proper mass, possibly calculated from Solidworks? -->
+        <inertia ixx="1.0" ixy="0.0" ixz="0.0" iyy="1.0" iyz="0.0" izz="1.0"/> <!-- TODO: Update with proper inertial values, possibly calculated from Solidworks? -->
+      </inertial>
+    </link>
+    <joint name="${name}_joint" type="continuous">
+      <parent link="base_link"/>
+      <child link="${name}"/><!--rpy="0 0 ${pi/2}"-->
+      <origin xyz="${fb*base_length/2 - 8*fb*itom} ${lr*base_width/2 + lr*wheel_width} ${-base_height/2}"/>
+      <axis xyz="0 1 0"/>
+      <limit effort="10000000.0"  velocity="10000"/>
+      <dynamics damping="0.7"/>
+    </joint>
+    <transmission name="${name}_tran">
+      <type>transmission_interface/SimpleTransmission</type>
+      <joint name="${name}_joint">
+        <hardwareInterface>hardware_interface/EffortJointInterface</hardwareInterface>
+      </joint>
+      <actuator name="${name}_motor">
+        <hardwareInterface>hardware_interface/EffortJointInterface</hardwareInterface>
+        <mechanicalReduction>1</mechanicalReduction>
+      </actuator>
+    </transmission>
+  </xacro:macro>
   <link name="god" /> <!-- This is necessary because Gazebo complains about the base link having inertia, for some reason -->
   <link name="base_link" >
@@ -18,8 +61,12 @@
     </collision>
     <inertial>
-      <mass value="250"/>
-      <inertia ixx="1.0" ixy="0.0" ixz="0.0" iyy="1.0" iyz="0.0" izz="1.0"/>
+      <mass value="250"/> <!-- TODO: Update with proper mass, possibly calculated from Solidworks? -->
+      <inertia ixx="1.0" ixy="0.0" ixz="0.0" iyy="1.0" iyz="0.0" izz="1.0"/> <!-- TODO: Update with proper inertial values, possibly calculated from Solidworks? -->
     </inertial>
   </link>
+  <xacro:wheel name="wheel_fr" fb="1" lr="-1" />
+  <xacro:wheel name="wheel_fl" fb="1" lr="1" />
+  <xacro:wheel name="wheel_rr" fb="-1" lr="-1" />
+  <xacro:wheel name="wheel_rl" fb="-1" lr="1" />
   <joint name="god_to_base" type="fixed">
     <parent link="god" />

Commit message: Added a skid steer controller and model tweaks

File: exc_description/urdf/exc.xacro (robot description, xacro)
@@ -5,5 +5,5 @@
   <xacro:property name="base_length" value="${58*itom}"/> <!-- Max val: 50" bare minimum -->
   <xacro:property name="base_height" value="${2*itom}"/> <!-- BS'd this number, total random guess -->
-  <xacro:property name="wheel_radius" value="${16*itom}"/>
+  <xacro:property name="wheel_radius" value="${6*itom}"/>
   <xacro:property name="wheel_width" value="${6*itom}"/>
   <xacro:include filename="$(find exc_description)/urdf/exc.gazebo" />
@@ -26,5 +26,5 @@
         <origin xyz="0 ${wheel_width/2} 0" rpy="0 0 0"/>
         <mass value="500"/> <!-- TODO: Update with proper mass, possibly calculated from Solidworks? -->
-        <inertia ixx="1.0" ixy="0.0" ixz="0.0" iyy="1.0" iyz="0.0" izz="1.0"/> <!-- TODO: Update with proper inertial values, possibly calculated from Solidworks? -->
+        <inertia ixx="1000.0" ixy="0.0" ixz="0.0" iyy="1000.0" iyz="0.0" izz="1000.0"/> <!-- TODO: Update with proper inertial values, possibly calculated from Solidworks? -->
       </inertial>
     </link>
@@ -32,7 +32,8 @@
       <parent link="base_link"/>
       <child link="${name}"/><!--rpy="0 0 ${pi/2}"-->
-      <origin xyz="${fb*base_length/2 - 8*fb*itom} ${lr*base_width/2 + lr*wheel_width} ${-base_height/2}"/>
+      <!-- TODO: Settle to more reasonable numbers -->
+      <origin xyz="${fb*base_length/2 - 16*fb*itom} ${lr*base_width/2 + lr*wheel_width} ${-base_height/2}"/>
       <axis xyz="0 1 0"/>
-      <limit effort="10000000.0"  velocity="10000"/>
+      <limit effort="100.0"  velocity="100.0"/>
       <dynamics damping="0.7"/>
     </joint>
@@ -45,4 +46,5 @@
         <hardwareInterface>hardware_interface/EffortJointInterface</hardwareInterface>
         <mechanicalReduction>1</mechanicalReduction>
+        <motorTorqueConstant>1</motorTorqueConstant>
       </actuator>
     </transmission>
@@ -62,5 +64,5 @@
     <inertial>
       <mass value="250"/> <!-- TODO: Update with proper mass, possibly calculated from Solidworks? -->
-      <inertia ixx="1.0" ixy="0.0" ixz="0.0" iyy="1.0" iyz="0.0" izz="1.0"/> <!-- TODO: Update with proper inertial values, possibly calculated from Solidworks? -->
+      <inertia ixx="1000.0" ixy="0.0" ixz="0.0" iyy="1000.0" iyz="0.0" izz="1000.0"/> <!-- TODO: Update with proper inertial values, possibly calculated from Solidworks? -->
     </inertial>
   </link>
@@ -72,4 +74,5 @@
     <parent link="god" />
     <child link="base_link" />
+    <origin xyz="0 0 0" />
   </joint>
 </robot>

Commit message: Added control package, fixed a build issue

File: exc_description/urdf/exc.xacro (robot description, xacro)
@@ -26,5 +26,5 @@
         <origin xyz="0 ${wheel_width/2} 0" rpy="0 0 0"/>
         <mass value="500"/> <!-- TODO: Update with proper mass, possibly calculated from Solidworks? -->
-        <inertia ixx="1000.0" ixy="0.0" ixz="0.0" iyy="1000.0" iyz="0.0" izz="1000.0"/> <!-- TODO: Update with proper inertial values, possibly calculated from Solidworks? -->
+        <inertia ixx="10.0" ixy="0.0" ixz="0.0" iyy="10.0" iyz="0.0" izz="10.0"/> <!-- TODO: Update with proper inertial values, possibly calculated from Solidworks? -->
       </inertial>
     </link>
@@ -63,6 +63,6 @@
     </collision>
     <inertial>
-      <mass value="250"/> <!-- TODO: Update with proper mass, possibly calculated from Solidworks? -->
-      <inertia ixx="1000.0" ixy="0.0" ixz="0.0" iyy="1000.0" iyz="0.0" izz="1000.0"/> <!-- TODO: Update with proper inertial values, possibly calculated from Solidworks? -->
+      <mass value="50"/> <!-- TODO: Update with proper mass, possibly calculated from Solidworks? -->
+      <inertia ixx="100.0" ixy="0.0" ixz="0.0" iyy="100.0" iyz="0.0" izz="100.0"/> <!-- TODO: Update with proper inertial values, possibly calculated from Solidworks? -->
     </inertial>
   </link>

Commit message: Cosmetic change adding tank treads

File: exc_description/urdf/exc.xacro (robot description, xacro)
@@ -33,5 +33,5 @@
       <child link="${name}"/><!--rpy="0 0 ${pi/2}"-->
       <!-- TODO: Settle to more reasonable numbers -->
-      <origin xyz="${fb*base_length/2 - 16*fb*itom} ${lr*base_width/2 + lr*wheel_width} ${-base_height/2}"/>
+      <origin xyz="${fb*base_length/2 - 16*fb*itom} ${lr*base_width/2 + lr*wheel_width/2} ${-base_height/2}"/>
       <axis xyz="0 1 0"/>
       <limit effort="100.0"  velocity="100.0"/>
@@ -50,4 +50,54 @@
     </transmission>
   </xacro:macro>
+  <link name="tread_left" >
+    <visual>
+      <geometry>
+        <cylinder radius="${wheel_radius}" length="${wheel_width}"/>
+      </geometry>
+      <origin xyz="${base_length/2-wheel_radius} 0 ${-wheel_width/2}" />
+    </visual>
+    <visual>
+      <geometry>
+        <cylinder radius="${wheel_radius}" length="${wheel_width}"/>
+      </geometry>
+      <origin xyz="${-base_length/2+wheel_radius} 0 ${-wheel_width/2}" />
+    </visual>
+    <visual>
+      <geometry>
+        <box size="${base_length-2*wheel_radius} ${2*wheel_radius} ${wheel_width}" />
+      </geometry>
+      <origin xyz="0 0 ${-wheel_width/2}" />
+    </visual>
+  </link>
+  <link name="tread_right" >
+    <visual>
+      <geometry>
+        <cylinder radius="${wheel_radius}" length="${wheel_width}"/>
+      </geometry>
+      <origin xyz="${base_length/2-wheel_radius} 0 ${wheel_width/2}" />
+    </visual>
+    <visual>
+      <geometry>
+        <cylinder radius="${wheel_radius}" length="${wheel_width}"/>
+      </geometry>
+      <origin xyz="${-base_length/2+wheel_radius} 0 ${wheel_width/2}" />
+    </visual>
+    <visual>
+      <geometry>
+        <box size="${base_length-2*wheel_radius} ${2*wheel_radius} ${wheel_width}" />
+      </geometry>
+      <origin xyz="0 0 ${wheel_width/2}" />
+    </visual>
+  </link>
+  <joint name="left_tread_to_base" type="fixed">
+    <parent link="base_link" />
+    <child link="tread_left" />
+    <origin xyz="0 ${base_width/2} ${-base_height/2}" rpy="${pi/2} 0 0" />
+  </joint>
+    <joint name="right_tread_to_base" type="fixed">
+      <parent link="base_link" />
+      <child link="tread_right" />
+      <origin xyz="0 ${-base_width/2} ${-base_height/2}" rpy="${pi/2} 0 0" />
+    </joint>
   <link name="god" /> <!-- This is necessary because Gazebo complains about the base link having inertia, for some reason -->
   <link name="base_link" >

Commit message: Added an arm turntable with control in the DS app
Use < and > (comma and period) to rotate the turntable by 15 deg/press

File: exc_description/urdf/exc.xacro (robot description, xacro)
@@ -8,4 +8,5 @@
   <xacro:property name="wheel_width" value="${6*itom}"/>
   <xacro:include filename="$(find exc_description)/urdf/exc.gazebo" />
+  <!-- fold Base Robot -->
   <!-- A macro for creating a wheel with a link, joint, and transmission -->
   <xacro:macro name="wheel" params="name fb lr">
@@ -95,9 +96,9 @@
     <origin xyz="0 ${base_width/2} ${-base_height/2}" rpy="${pi/2} 0 0" />
   </joint>
-    <joint name="right_tread_to_base" type="fixed">
-      <parent link="base_link" />
-      <child link="tread_right" />
-      <origin xyz="0 ${-base_width/2} ${-base_height/2}" rpy="${pi/2} 0 0" />
-    </joint>
+  <joint name="right_tread_to_base" type="fixed">
+    <parent link="base_link" />
+    <child link="tread_right" />
+    <origin xyz="0 ${-base_width/2} ${-base_height/2}" rpy="${pi/2} 0 0" />
+  </joint>
   <link name="god" /> <!-- This is necessary because Gazebo complains about the base link having inertia, for some reason -->
   <link name="base_link" >
@@ -126,3 +127,41 @@
     <origin xyz="0 0 0" />
   </joint>
+  <!-- /fold -->
+  <link name="turntable">
+    <visual>
+      <geometry>
+        <cylinder radius="${base_width/3}" length="${6*itom}" />
+      </geometry>
+      <origin xyz="0 0 ${3*itom}" />
+    </visual>
+    <collision>
+      <geometry>
+        <cylinder radius="${base_width/3}" length="${12*itom}" />
+        <origin xyz="0 0 ${3*itom}" />
+      </geometry>
+    </collision>
+    <inertial>
+      <mass value="50"/> <!-- TODO: Update with proper mass, possibly calculated from Solidworks? -->
+      <inertia ixx="100.0" ixy="0.0" ixz="0.0" iyy="100.0" iyz="0.0" izz="100.0"/> <!-- TODO: Update with proper inertial values, possibly calculated from Solidworks? -->
+    </inertial>
+  </link>
+  <joint name="turn_to_base" type="continuous">
+    <parent link="base_link" />
+    <child link="turntable" />
+    <origin xyz="${base_length/2-base_width/3-3*itom} 0 ${base_height/2}" />
+    <axis xyz="0 0 1" />
+    <limit effort="100.0"  velocity="0.25"/>
+    <dynamics damping="0.7"/>
+  </joint>
+  <transmission name="turntable_tran">
+    <type>transmission_interface/SimpleTransmission</type>
+    <joint name="turn_to_base">
+      <hardwareInterface>hardware_interface/EffortJointInterface</hardwareInterface>
+    </joint>
+    <actuator name="turntable_motor">
+      <hardwareInterface>hardware_interface/EffortJointInterface</hardwareInterface>
+      <mechanicalReduction>1</mechanicalReduction>
+      <motorTorqueConstant>1</motorTorqueConstant>
+    </actuator>
+  </transmission>
 </robot>

Commit message: Added the lower and upper arm segments and control

File: exc_description/urdf/exc.xacro (robot description, xacro)
@@ -128,4 +128,5 @@
   </joint>
   <!-- /fold -->
+  <!-- fold Turntable -->
   <link name="turntable">
     <visual>
@@ -137,5 +138,5 @@
     <collision>
       <geometry>
-        <cylinder radius="${base_width/3}" length="${12*itom}" />
+        <cylinder radius="${base_width/3}" length="${6*itom}" />
         <origin xyz="0 0 ${3*itom}" />
       </geometry>
@@ -151,5 +152,5 @@
     <origin xyz="${base_length/2-base_width/3-3*itom} 0 ${base_height/2}" />
     <axis xyz="0 0 1" />
-    <limit effort="100.0"  velocity="0.25"/>
+    <limit effort="1000.0"  velocity="0.25"/>
     <dynamics damping="0.7"/>
   </joint>
@@ -160,4 +161,79 @@
     </joint>
     <actuator name="turntable_motor">
+      <hardwareInterface>hardware_interface/EffortJointInterface</hardwareInterface>
+      <mechanicalReduction>1</mechanicalReduction>
+      <motorTorqueConstant>1</motorTorqueConstant>
+    </actuator>
+  </transmission>
+  <!-- /fold -->
+  <link name="arm_lower">
+    <visual>
+      <geometry>
+        <box size="${4*itom} ${4*itom} ${36*itom}" />
+      </geometry>
+      <origin xyz="0 0 ${18*itom}" />
+    </visual>
+    <collision>
+      <geometry>
+        <box size="${4*itom} ${4*itom} ${36*itom}" />
+      </geometry>
+      <origin xyz="0 0 ${18*itom}" />
+    </collision>
+    <inertial>
+      <mass value="50"/> <!-- TODO: Update with proper mass, possibly calculated from Solidworks? -->
+      <inertia ixx="100.0" ixy="0.0" ixz="0.0" iyy="100.0" iyz="0.0" izz="100.0"/> <!-- TODO: Update with proper inertial values, possibly calculated from Solidworks? -->
+    </inertial>
+  </link>
+  <joint name="lower_to_turn" type="revolute">
+    <parent link="turntable" />
+    <child link="arm_lower" />
+    <axis xyz="0 1 0" />
+    <origin xyz="0 0 ${6*itom}" />
+    <limit effort="500.0"  velocity="0.25" lower="${-pi/6}" upper="${3*pi/8}"/>
+    <dynamics damping="5.0"/>
+  </joint>
+  <transmission name="lower_arm_tran">
+    <type>transmission_interface/SimpleTransmission</type>
+    <joint name="lower_to_turn">
+      <hardwareInterface>hardware_interface/EffortJointInterface</hardwareInterface>
+    </joint>
+    <actuator name="lower_motor">
+      <hardwareInterface>hardware_interface/EffortJointInterface</hardwareInterface>
+      <mechanicalReduction>1</mechanicalReduction>
+      <motorTorqueConstant>1</motorTorqueConstant>
+    </actuator>
+  </transmission>
+  <link name="arm_upper">
+    <visual>
+      <geometry>
+        <box size="${4*itom} ${4*itom} ${36*itom}" />
+      </geometry>
+      <origin xyz="0 0 ${18*itom}" />
+    </visual>
+    <collision>
+      <geometry>
+        <box size="${4*itom} ${4*itom} ${36*itom}" />
+      </geometry>
+      <origin xyz="0 0 ${18*itom}" />
+    </collision>
+    <inertial>
+      <mass value="50"/> <!-- TODO: Update with proper mass, possibly calculated from Solidworks? -->
+      <inertia ixx="100.0" ixy="0.0" ixz="0.0" iyy="100.0" iyz="0.0" izz="100.0"/> <!-- TODO: Update with proper inertial values, possibly calculated from Solidworks? -->
+    </inertial>
+  </link>
+  <joint name="upper_to_lower" type="revolute">
+    <parent link="arm_lower" />
+    <child link="arm_upper" />
+    <axis xyz="0 1 0" />
+    <origin xyz="0 0 ${36*itom}" />
+    <limit effort="500.0"  velocity="0.25" lower="0.0" upper="${3*pi/8}"/>
+    <dynamics damping="5.0"/>
+  </joint>
+  <transmission name="upper_arm_tran">
+    <type>transmission_interface/SimpleTransmission</type>
+    <joint name="upper_to_lower">
+      <hardwareInterface>hardware_interface/EffortJointInterface</hardwareInterface>
+    </joint>
+    <actuator name="upper_motor">
       <hardwareInterface>hardware_interface/EffortJointInterface</hardwareInterface>
       <mechanicalReduction>1</mechanicalReduction>

Commit message: fixed jumpy IMU, bug in RVIX

File: exc_description/urdf/exc.xacro (robot description, xacro)
@@ -126,3 +126,61 @@
     <origin xyz="0 0 0" />
   </joint>
+ <joint name="imu_joint" type="fixed">
+      <axis xyz="0 0 0"/>
+      <origin xyz="0 0 0.0512"/>
+      <parent link="base_link"/>
+      <child link="imu_link"/>
+  </joint>
+  <link name="imu_link">
+      <inertial>
+          <mass value="0.05"/>
+          <origin rpy="0 0 0" xyz="0 0 .05"/>
+          <inertia ixx="0.05" ixy="0" ixz="0" iyy="0.05" iyz="0" izz="0.05"/>
+      </inertial>
+      <visual>
+          <origin rpy="0 0 0" xyz="0 0 0.05"/>
+          <geometry>
+              <box size="0.1 0.1 0.1"/>
+          </geometry>
+      </visual>
+      <collision>
+          <origin rpy="0 0 0" xyz="0 0 .05"/>
+          <geometry>
+              <box size=".1 .1 .1"/>
+          </geometry>
+      </collision>
+  </link>
+  <gazebo>
+      <plugin name="imu_plugin" filename="libgazebo_ros_imu.so">
+          <robotNamespace>/exc</robotNamespace>
+          <alwaysOn>true</alwaysOn>
+          <xyzOffset>0 0 .05</xyzOffset>
+          <bodyName>imu_link</bodyName>
+          <topicName>imu</topicName>
+          <serviceName>imu_service</serviceName>
+          <frameName>imu_link</frameName>
+          <gaussianNoise>0.05</gaussianNoise>
+          <updateRate>20.0</updateRate>
+      </plugin>
+</gazebo>
+<!--  <gazebo reference="imu_link">
+    <gravity>true</gravity>
+   <sensor name="imu_sensor" type="imu">
+      <always_on>true</always_on>
+      <update_rate>50</update_rate>
+      <visualize>true</visualize>
+      <topic>imuTest</topic>
+      <plugin filename="libgazebo_ros_imu_sensor.so" name="imu_plugin">
+        <robotNamespace>/exc</robotNamespace>
+        <topicName>imu</topicName>
+        <bodyName>imu_link</bodyName>
+        <updateRateHZ>50.0</updateRateHZ>
+        <gaussianNoise>0.00</gaussianNoise>
+        <xyzOffset>0 0 0.05</xyzOffset>
+        <rpyOffset>0 0 0</rpyOffset>
+        <frameName>imu_link</frameName>
+      </plugin>
+      <pose>0 0 0 0 0 0</pose>
+    </sensor>
+</gazebo>-->
 </robot>

Commit message: Added the MoveIt package and basic implementation

File: exc_description/urdf/exc.xacro (robot description, xacro)
@@ -241,3 +241,15 @@
     </actuator>
   </transmission>
+  <link name="arm_end" >
+    <visual>
+      <geometry>
+        <box size="0.1 0.1 0.1" />
+      </geometry>
+    </visual>
+  </link>
+  <joint name="end_to_arm" type="fixed">
+    <parent link="arm_upper" />
+    <child link="arm_end" />
+    <origin xyz="0 0 ${36*itom}" />
+  </joint>
 </robot>

Commit message: Resolved MoveIt issues, now fully functional

File: exc_description/urdf/exc.xacro (robot description, xacro)
@@ -152,5 +152,5 @@
     <origin xyz="${base_length/2-base_width/3-3*itom} 0 ${base_height/2}" />
     <axis xyz="0 0 1" />
-    <limit effort="1000.0"  velocity="0.25"/>
+    <limit effort="10000.0"  velocity="0.25"/>
     <dynamics damping="0.7"/>
   </joint>
@@ -190,5 +190,5 @@
     <axis xyz="0 1 0" />
     <origin xyz="0 0 ${6*itom}" />
-    <limit effort="500.0"  velocity="0.25" lower="${-pi/6}" upper="${3*pi/8}"/>
+    <limit effort="10000.0"  velocity="0.25" lower="${-pi/6}" upper="${3*pi/8}"/>
     <dynamics damping="5.0"/>
   </joint>
@@ -227,5 +227,5 @@
     <axis xyz="0 1 0" />
     <origin xyz="0 0 ${36*itom}" />
-    <limit effort="500.0"  velocity="0.25" lower="0.0" upper="${3*pi/8}"/>
+    <limit effort="10000.0"  velocity="0.25" lower="0.0" upper="${3*pi/8}"/>
     <dynamics damping="5.0"/>
   </joint>
@@ -244,12 +244,31 @@
     <visual>
       <geometry>
-        <box size="0.1 0.1 0.1" />
-      </geometry>
-    </visual>
-  </link>
-  <joint name="end_to_arm" type="fixed">
+        <box size="${12*itom} ${12*itom} ${4*itom}" />
+      </geometry>
+      <origin xyz="${6*itom} 0 0" />
+    </visual>
+    <inertial>
+      <mass value="50"/> <!-- TODO: Update with proper mass, possibly calculated from Solidworks? -->
+      <inertia ixx="100.0" ixy="0.0" ixz="0.0" iyy="100.0" iyz="0.0" izz="100.0"/> <!-- TODO: Update with proper inertial values, possibly calculated from Solidworks? -->
+    </inertial>
+  </link>
+  <joint name="end_to_arm" type="revolute">
     <parent link="arm_upper" />
     <child link="arm_end" />
     <origin xyz="0 0 ${36*itom}" />
-  </joint>
+    <axis xyz="0 1 0" />
+    <limit effort="10000.0" velocity="0.25" lower="${-3*pi/8}" upper="${pi/4}" />
+    <dynamics damping="5.0"/>
+  </joint>
+  <transmission name="arm_end_tran">
+    <type>transmission_interface/SimpleTransmission</type>
+    <joint name="end_to_arm">
+      <hardwareInterface>hardware_interface/EffortJointInterface</hardwareInterface>
+    </joint>
+    <actuator name="end_motor">
+      <hardwareInterface>hardware_interface/EffortJointInterface</hardwareInterface>
+      <mechanicalReduction>1</mechanicalReduction>
+      <motorTorqueConstant>1</motorTorqueConstant>
+    </actuator>
+  </transmission>
 </robot>

Commit message: Added a test lidar to the robot
Settings are approximately the same as our lidar we'll be purchasing.

File: exc_description/urdf/exc.xacro (robot description, xacro)
@@ -121,4 +121,26 @@
   <xacro:wheel name="wheel_rr" fb="-1" lr="-1" />
   <xacro:wheel name="wheel_rl" fb="-1" lr="1" />
+  <link name="laser_link" >
+    <visual>
+      <geometry>
+        <box size="${itom} ${itom} ${itom}" />
+      </geometry>
+    </visual>
+    <collision>
+      <geometry>
+        <box size="${itom} ${itom} ${itom}" />
+      </geometry>
+    </collision>
+    <inertial>
+      <mass value="1e-5" />
+      <origin xyz="0 0 0" rpy="0 0 0"/>
+      <inertia ixx="1e-6" ixy="0" ixz="0" iyy="1e-6" iyz="0" izz="1e-6" />
+    </inertial>
+  </link>
+  <joint name="laser_to_base" type="fixed">
+    <parent link="base_link" />
+    <child link="laser_link" />
+    <origin xyz="${base_length/2} 0 ${12*itom}" />
+  </joint>
   <joint name="god_to_base" type="fixed">
     <parent link="god" />
