Commit message: Tested laser_filter on the robot

File: exc_description/urdf/exc.xacro (robot description, xacro)
@@ -138,8 +138,30 @@
     </inertial>
   </link>
+  <link name="annoying_robot_part_that_gets_in_the_way_of_everything" >
+    <visual>
+      <geometry>
+        <box size="${6*itom} ${6*itom} ${18*itom}" />
+      </geometry>
+    </visual>
+    <collision>
+      <geometry>
+        <box size="${6*itom} ${6*itom} ${18*itom}" />
+      </geometry>
+    </collision>
+    <inertial>
+      <mass value="1e-5" />
+      <origin xyz="0 0 0" rpy="0 0 0"/>
+      <inertia ixx="1e-6" ixy="0" ixz="0" iyy="1e-6" iyz="0" izz="1e-6" />
+    </inertial>
+  </link>
   <joint name="laser_to_base" type="fixed">
     <parent link="base_link" />
     <child link="laser_link" />
     <origin xyz="${base_length/2} 0 ${12*itom}" />
+  </joint>
+  <joint name="annoyance_to_base" type="fixed">
+    <parent link="base_link" />
+    <child link="annoying_robot_part_that_gets_in_the_way_of_everything" />
+    <origin xyz="${-base_length/2} 0 ${base_height + 6*itom}" />
   </joint>
   <joint name="god_to_base" type="fixed">

Commit message: Added a basic stereo camera (Kinect)
Parameters are untuned for now (FOV, point density, etc.), I'll leave
this to the members working with this prototype more. Also added a
starting implementation of rtabmap for testing the autonomous navigation

File: exc_description/urdf/exc.xacro (robot description, xacro)
@@ -126,3 +126,25 @@
     <origin xyz="0 0 0" />
   </joint>
+  <link name="kinect_link" >
+    <visual>
+      <geometry>
+        <box size="${itom} ${itom} ${itom}" />
+      </geometry>
+    </visual>
+    <collision>
+      <geometry>
+        <box size="${itom} ${itom} ${itom}" />
+      </geometry>
+    </collision>
+    <inertial>
+      <mass value="1e-5" />
+      <origin xyz="0 0 0" rpy="0 0 0"/>
+      <inertia ixx="1e-6" ixy="0" ixz="0" iyy="1e-6" iyz="0" izz="1e-6" />
+    </inertial>
+  </link>
+  <joint name="kinect_to_base" type="fixed">
+    <parent link="base_link" />
+    <child link="kinect_link" />
+    <origin xyz="${base_length/2} 0 ${12*itom}" />
+  </joint>
 </robot>

Commit message: Added the arm joint controller
Had to tweak a large number of things. Discovered that I can't have multiple controller "launcher" nodes, it doesn't like it (or at least how I was trying to do it), so I made one overall "controller launcher" and "hardware interface" that does both the arm and drivebase. This isn't really an issue, it's just a bit less modularity.

File: exc_description/urdf/exc.xacro (robot description, xacro)
@@ -126,3 +126,38 @@
     <origin xyz="0 0 0" />
   </joint>
+  <link name="arm">
+    <visual>
+      <geometry>
+        <box size="${6*itom} ${6*itom} ${24*itom}" />
+      </geometry>
+      <origin xyz="0 0 ${12*itom}" />
+    </visual>
+    <collision>
+      <geometry>
+        <box size="${6*itom} ${6*itom} ${24*itom}" />
+      </geometry>
+      <origin xyz="0 0 ${12*itom}" />
+    </collision>
+    <inertial>
+      <mass value="50"/> <!-- TODO: Update with proper mass, possibly calculated from Solidworks? -->
+      <inertia ixx="100.0" ixy="0.0" ixz="0.0" iyy="100.0" iyz="0.0" izz="100.0"/> <!-- TODO: Update with proper inertial values, possibly calculated from Solidworks? -->
+    </inertial>
+  </link>
+  <joint name="arm_joint" type="revolute">
+    <parent link="base_link" />
+    <child link="arm" />
+    <origin xyz="${base_length/2} 0 ${base_height/2}" rpy="0 0 ${pi/2}" />
+    <limit effort="50.0" velocity="50.0" lower="0.0" upper="${pi/2}" />
+  </joint>
+  <transmission name="arm_tran">
+    <type>transmission_interface/SimpleTransmission</type>
+    <joint name="arm_joint">
+      <hardwareInterface>hardware_interface/EffortJointInterface</hardwareInterface>
+    </joint>
+    <actuator name="arm_motor">
+      <hardwareInterface>hardware_interface/EffortJointInterface</hardwareInterface>
+      <mechanicalReduction>1</mechanicalReduction>
+      <motorTorqueConstant>1</motorTorqueConstant>
+    </actuator>
+  </transmission>
 </robot>

Commit message: Fixed drive flip and potentiometer reading

File: exc_description/urdf/exc.xacro (robot description, xacro)
@@ -148,5 +148,5 @@
     <child link="arm" />
     <origin xyz="${base_length/2} 0 ${base_height/2}" rpy="0 0 ${pi/2}" />
-    <limit effort="50.0" velocity="50.0" lower="0.0" upper="${pi/2}" />
+    <limit effort="50.0" velocity="50.0" lower="${70*pi/180}" upper="${140*pi/180}" />
   </joint>
   <transmission name="arm_tran">

Commit message: added stereo camera plugin

File: exc_description/urdf/exc.xacro (robot description, xacro)
@@ -8,4 +8,5 @@
   <xacro:property name="wheel_width" value="${6*itom}"/>
   <xacro:include filename="$(find exc_description)/urdf/exc.gazebo" />
+  <!--DRIVEBASE-->
   <!-- A macro for creating a wheel with a link, joint, and transmission -->
   <xacro:macro name="wheel" params="name fb lr">
@@ -100,4 +101,9 @@
       <origin xyz="0 ${-base_width/2} ${-base_height/2}" rpy="${pi/2} 0 0" />
     </joint>
+  <xacro:wheel name="wheel_fr" fb="1" lr="-1" />
+  <xacro:wheel name="wheel_fl" fb="1" lr="1" />
+  <xacro:wheel name="wheel_rr" fb="-1" lr="-1" />
+  <xacro:wheel name="wheel_rl" fb="-1" lr="1" />
+  <!--GOD-->
   <link name="god" /> <!-- This is necessary because Gazebo complains about the base link having inertia, for some reason -->
   <link name="base_link" >
@@ -117,8 +123,4 @@
     </inertial>
   </link>
-  <xacro:wheel name="wheel_fr" fb="1" lr="-1" />
-  <xacro:wheel name="wheel_fl" fb="1" lr="1" />
-  <xacro:wheel name="wheel_rr" fb="-1" lr="-1" />
-  <xacro:wheel name="wheel_rl" fb="-1" lr="1" />
   <joint name="god_to_base" type="fixed">
     <parent link="god" />
@@ -126,3 +128,31 @@
     <origin xyz="0 0 0" />
   </joint>
+  <!--STEREO CAMERA-->
+  <xacro:property name="camera_size" value="0.05" /> <!-- Size of square 'camera' box -->
+  <joint name="camera_joint" type="fixed">
+    <origin xyz="${base_length/2} 0 ${base_height/2}" rpy="0 0 0"/>
+    <parent link="base_link"/>
+    <child link="camera_link"/>
+  </joint>
+  <!-- Camera -->
+  <link name="camera_link">
+    <collision>
+      <origin xyz="-${camera_size/2} 0 ${camera_size/2}" rpy="0 0 0"/>
+      <geometry>
+      <box size="${camera_size} ${camera_size} ${camera_size}"/>
+      </geometry>
+    </collision>
+    <visual>
+      <origin xyz="-${camera_size/2} 0 ${camera_size/2}" rpy="0 0 0"/>
+      <geometry>
+    <box size="${camera_size} ${camera_size} ${camera_size}"/>
+      </geometry>
+      <material name="red"/>
+    </visual>
+    <inertial>
+      <mass value="1e-5" />
+      <origin xyz="-${camera_size/2} 0 ${camera_size/2}" rpy="0 0 0"/>
+      <inertia ixx="1e-6" ixy="0" ixz="0" iyy="1e-6" iyz="0" izz="1e-6" />
+    </inertial>
+  </link>
 </robot>
