Commit message: added imus

File: tfr_description/urdf/model.xacro (robot description, xacro)
@@ -95,9 +95,9 @@
     <origin xyz="0 ${base_width/2} ${-base_height/2}" rpy="${pi/2} 0 0" />
   </joint>
-    <joint name="right_tread_to_base" type="fixed">
-      <parent link="base_link" />
-      <child link="tread_right" />
-      <origin xyz="0 ${-base_width/2} ${-base_height/2}" rpy="${pi/2} 0 0" />
-    </joint>
+  <joint name="right_tread_to_base" type="fixed">
+    <parent link="base_link" />
+    <child link="tread_right" />
+    <origin xyz="0 ${-base_width/2} ${-base_height/2}" rpy="${pi/2} 0 0" />
+  </joint>
   <xacro:wheel name="wheel_fr" fb="1" lr="-1" />
   <xacro:wheel name="wheel_fl" fb="1" lr="1" />
@@ -138,5 +138,5 @@
       <origin xyz="-${camera_size/2} 0 ${camera_size/2}" rpy="0 0 0"/>
       <geometry>
-      <box size="${camera_size} ${camera_size} ${camera_size}"/>
+        <box size="${camera_size} ${camera_size} ${camera_size}"/>
       </geometry>
     </collision>
@@ -144,5 +144,5 @@
       <origin xyz="-${camera_size/2} 0 ${camera_size/2}" rpy="0 0 0"/>
       <geometry>
-    <box size="${camera_size} ${camera_size} ${camera_size}"/>
+        <box size="${camera_size} ${camera_size} ${camera_size}"/>
       </geometry>
       <material name="red"/>
@@ -154,3 +154,30 @@
     </inertial>
   </link>
+  <!--IMU-->
+  <xacro:property name="imu_size" value="0.05" /> <!-- Size of square 'camera' box -->
+  <joint name="imu_joint" type="fixed">
+    <axis xyz="0 0 0"/>
+    <origin xyz="0 0 ${base_height/2}"/>
+    <parent link="base_link"/>
+    <child link="imu_link"/>
+  </joint>
+  <link name="imu_link">
+    <inertial>
+      <mass value="1e-5" />
+      <origin rpy="0 0 0" xyz="0 0 ${base_height/2}"/>
+      <inertia ixx="1e-6" ixy="0" ixz="0" iyy="1e-6" iyz="0" izz="1e-6" />
+    </inertial>
+    <visual>
+      <origin rpy="0 0 0" xyz="0 0 ${base_height/2}"/>
+      <geometry>
+        <box size="${imu_size} ${imu_size} ${imu_size}"/>
+      </geometry>
+    </visual>
+    <collision>
+      <origin rpy="0 0 0" xyz="0 0 ${base_height/2}"/>
+      <geometry>
+        <box size="${imu_size} ${imu_size} ${imu_size}"/>
+      </geometry>
+    </collision>
+  </link>
 </robot>

File: tfr_description/urdf/sensors.xacro (robot description, xacro)
@@ -42,3 +42,27 @@
     </sensor>
   </gazebo>
+  <gazebo>
+    <plugin name="imu_plugin" filename="libgazebo_ros_imu.so">
+      <robotNamespace>/</robotNamespace>
+      <alwaysOn>true</alwaysOn>
+      <bodyName>imu_link</bodyName>
+      <topicName>/sensors/mti/imu/data</topicName>
+      <serviceName>/sensors/mti/imu/data_srv</serviceName>
+      <frameName>imu_link</frameName>
+      <gaussianNoise>0.02</gaussianNoise>
+      <updateRate>60.0</updateRate>
+    </plugin>
+  </gazebo>
+  <gazebo>
+    <plugin name="imu_plugin" filename="libgazebo_ros_imu.so">
+      <robotNamespace>/</robotNamespace>
+      <alwaysOn>true</alwaysOn>
+      <bodyName>camera_link</bodyName>
+      <topicName>/sensors/duo_3d/imu/data_raw</topicName>
+      <serviceName>/sensors/duo_3d/imu/data_raw_srv</serviceName>
+      <frameName>camera_link</frameName>
+      <gaussianNoise>0.05</gaussianNoise>
+      <updateRate>60.0</updateRate>
+    </plugin>
+  </gazebo>
 </robot>
